File: hardware/Processor Board.sch (EAGLE design)
At the start: 0 parts

Commit message: Add bitmaps and python code to turn them into valid C++
This python is an abomination 🙃🐍
Parts:
- added ANT: ANTENNA_CHIP2450AT43B100, _Antennas:ANTENNA_CHIP2450AT43B100
- added C1, C10, C11, C2, C4: .1µF, SparkFun-Passives:CAP0805
- added C12, C13: 12pF, SparkFun-Passives:CAP0805
- added C14: 4.7µF, SparkFun-Passives:CAP0805
- added C3: 1nF, SparkFun-Passives:CAP0805
- added C5: 47nF, SparkFun-Passives:CAP0805
- added C6: 2.2nf, SparkFun-Passives:CAP0805
- added C7: 3.9pF, SparkFun-Passives:CAP0805
- added C8: 1pF, SparkFun-Passives:CAP0805
- added C9: 1.5pF, SparkFun-Passives:CAP0805
- added D1: 250mA/100V, SparkFun-DiscreteSemi:DIODEBAS16
- added D2, D3, D4, D5: (no value), SparkFun-LED:LED1206
- added L1: 27nH, SparkFun-Passives:INDUCTOR0805
- added L2: 4.7nH, SparkFun-Passives:INDUCTOR0805
- added L3: 3.3nH, SparkFun-Passives:INDUCTOR0805
- added L4: 2.7nH, SparkFun-Passives:INDUCTOR0805
- added L5: 2.2nH, SparkFun-Passives:INDUCTOR0805
- added L6: ?, SparkFun-Passives:INDUCTOR0805
- added LCD1: LPH-7366, lph-7366:LPH-7366
- added LOGO1: OSHW-LOGOL-COPPER, SparkFun-Aesthetics:OSHW-LOGOL-COPPER
- added M1: (no value), SparkFun-Connectors:M021X02_NO_SILK
- added Q1: MPSA42, SparkFun-DiscreteSemi:TRANSISTOR_NPNMPSA42
- added R1, R2: 10kΩ, SparkFun-Passives:RESISTOR0805-RES
- added R3, R5: 270Ω, SparkFun-Passives:RESISTOR0805-RES
- added R4: 330Ω, SparkFun-Passives:RESISTOR0805-RES
- added S1: SPST.B3U-1000P(M)-B, omron:SPST.B3U-1000P(M)-B
- added TP1, TP2: TEST-POINT3, SparkFun-Passives:TEST-POINT3
- added U1: NRF51822, NordicSemi:NRF51822
- added U2: MMA8452Q, SparkFun-Sensors:MMA8452Q
- added U3: DS1307SO8, SparkFun-FreqCtrl:DS1307SO8
- added X1: CORTEX_DEBUGPTH, SparkFun-Connectors:CORTEX_DEBUGPTH
- added X2: Power, con-jst2:SM04B-SRSS-TB
- added X3: SM06B-SRSS-TB, con-jst2:SM06B-SRSS-TB
- added X4: HEADER-04-.05MM, _Connectors:HEADER-04-.05MM
- added X5: HEADER-06-.05IN, _Connectors:HEADER-06-.05IN
- added Y1: 16MHz, SparkFun-FreqCtrl:CRYSTALCRYSTAL-SMD-5X3-16MHZ
- added Y2: (no value), SparkFun-FreqCtrl:CRYSTAL32-SMD-MELF
Connections:
- new net ACC_INT1: U1.P0.13, U2.INT1
- new net ACC_INT2: U1.P0.14, U2.INT2
- new net ANT: ANT.ANT, L4.1, L5.1
- new net ANT1: L1.1, L2.2, U1.ANT1
- new net ANT2: C7.1, L2.1, U1.ANT2
- new net BACKLIGHT: R4.2, U1.P0.12
- new net BTN_BACK: S1.1, U1.P0.17
- new net BTN_DOWN: U1.P0.26, X3-2.S, X5.2
- new net BTN_LEFT: U1.P0.29, X3-5.S, X5.5
- new net BTN_RIGHT: U1.P0.28, X3-4.S, X5.4
- new net BTN_SELECT: U1.P0.25, X3-1.S, X5.1
- new net BTN_UP: U1.P0.27, X3-3.S, X5.3
- new net CHG: U1.P0.01, X2-3.S, X4.3
- new net F_1: C7.2, C8.2, L3.2
- new net F_2: C9.2, L3.1, L4.2, L6.1
- new net GND: C1.2, C10.2, C11.2, C12.1, C13.1, C14.2, C2.2, C3.2, C4.1, C5.2, C6.2, C8.1, C9.1, D2.C, D3.C, D4.C, D5.C, L5.2, L6.2, LCD1.GND, Q1.E, S1.2, TP2.1, U1.DIE_PAD, U1.VSS, U1.VSS_2, U1.VSS_3, U2.GND@0, U2.GND@1, U2.GND@2, U2.SA0, U3.GND, X1.GND@3, X1.GND@5, X1.GNDDTCT, X1.KEY, X2-4.S, X3-6.S, X4.4, X5.6
- new net IND: U1.P0.02, X2-2.S, X4.2
- new net LCD_CE: LCD1./SCE, U1.P0.04
- new net LCD_CLK: LCD1.SCLK, U1.P0.07
- new net LCD_DC: LCD1.D/C, U1.P0.05
- new net LCD_MOSI: LCD1.SDIN, U1.P0.06
- new net LCD_RST: LCD1./RES, U1.P0.03
- new net N$1: U1.SWDCLK, X1.SWDCLK/TCK
- new net N$10: Q1.B, R3.2
- new net N$11: C12.2, U1.XC2, Y1.2
- new net N$12: C13.2, U1.XC1, Y1.1
- new net N$13: U3.X1, Y2.2
- new net N$14: D1.A, M1.2, Q1.C
- new net N$15: M1.1, R5.1
- new net N$16: U3.X2, Y2.1
- new net N$17: D2.A, D3.A, D4.A, D5.A, R4.1
- new net N$2: C4.2, U1.DEC1
- new net N$3: U1.SWDIO/NRESET, X1.SWDIO/TMS
- new net N$4: C5.1, U1.DEC2
- new net N$6: C11.1, U2.BYP
- new net SCL: R1.1, U1.P0.16, U2.SCL, U3.SCL
- new net SDA: R2.1, U1.P0.15, U2.SDA, U3.SDA
- new net VCC: C1.1, C10.1, C14.1, C2.1, C3.1, D1.C, LCD1.OSC, LCD1.VDD, R1.2, R2.2, R5.2, TP1.1, U1.AVDD, U1.AVDD_2, U1.P0.00, U1.VDD, U1.VDD_2, U2.VDD, U2.VDDIO, U3.VCC, X1.VCC, X2-1.S, X4.1
- new net VDD_PA: C6.1, L1.2, U1.VDD_PA
- new net VIB: R3.1, U1.P0.21
Other:
- note added: "50Ω Impedence"
